File: SLAMP-WiFi/SLAMP-WiFi.sch (KiCad schematic (older format))
At the start: 2 parts

Commit message: Comenzando el desarrollo del conversor USB-UART
Parts:
- added C? (x2): 22p, symbol C
- added P?: CONN_01X04, symbol CONN_01X04
- added Y?: 12 MHz, symbol Crystal
Connections:
- net D+: now reaches U?.5 (D+)
- net D+: now also P?.2 (P2)
- net D-: now reaches U?.6 (D-)
- net D-: now also P?.3 (P3)
- net at U?.7 (XI): now also C?.1, Y?.1
- net at U?.8 (XO): now also C?.1, Y?.2
- new net GND: C?.2, C?.2, P?.1 (P1)
- new net VUSB: P?.4 (P4)
Other:
- moved on the sheet: U?
Changed lines of the file:
@@
 L ESP-12E U?
 U 1 1 5935D8C2
-P 6700 3100
-F 0 "U?" H 6700 3000 50  0000 C CNN
-F 1 "ESP-12F" H 6700 3200 50  0000 C CNN
-F 2 "" H 6700 3100 50  0001 C CNN
-F 3 "" H 6700 3100 50  0001 C CNN
-	1    6700 3100
+P 8600 2050
+F 0 "U?" H 8600 1950 50  0000 C CNN
+F 1 "ESP-12F" H 8600 2150 50  0000 C CNN
+F 2 "" H 8600 2050 50  0001 C CNN
+F 3 "" H 8600 2050 50  0001 C CNN
+	1    8600 2050
 	1    0    0    -1
 $EndComp
@@
 L CH340G U?
 U 1 1 5935DA35
-P 4150 3200
-F 0 "U?" H 4150 3760 60  0000 C CNN
-F 1 "CH340G" H 4150 2740 60  0000 C CNN
-F 2 "SOIC-16_N" H 4150 2650 40  0001 C CNN
-F 3 "" H 4150 3200 60  0000 C CNN
-	1    4150 3200
+P 3400 5400
+F 0 "U?" H 3400 5960 60  0000 C CNN
+F 1 "CH340G" H 3400 4940 60  0000 C CNN
+F 2 "SOIC-16_N" H 3400 4850 40  0001 C CNN
+F 3 "" H 3400 5400 60  0000 C CNN
+	1    3400 5400
 	1    0    0    -1
 $EndComp
+$Comp
+L CONN_01X04 P?
+U 1 1 594A46FC
+P 2300 3800
+F 0 "P?" H 2300 4050 50  0000 C CNN
+F 1 "CONN_01X04" V 2400 3800 50  0000 C CNN
+F 2 "" H 2300 3800 50  0001 C CNN
+F 3 "" H 2300 3800 50  0001 C CNN
+	1    2300 3800
+	-1   0    0    1
+$EndComp
+$Comp
+L GND #PWR?
+U 1 1 594A493D
+P 2600 4050
+F 0 "#PWR?" H 2600 3800 50  0001 C CNN
+F 1 "GND" H 2600 3900 50  0000 C CNN
+F 2 "" H 2600 4050 50  0001 C CNN
+F 3 "" H 2600 4050 50  0001 C CNN
+	1    2600 4050
+	1    0    0    -1
+$EndComp
+Text GLabel 2600 3500 1    39   Input ~ 0
+VUSB
+Text GLabel 2700 3850 2    39   Input ~ 0
+D+
+Text GLabel 2700 3750 2    39   Input ~ 0
+D-
+Text GLabel 2400 5400 0    39   Input ~ 0
+D+
+Text GLabel 2400 5500 0    39   Input ~ 0
+D-
+$Comp
+L Crystal Y?
+U 1 1 594A4A81
+P 2450 5950
+F 0 "Y?" H 2450 6100 50  0000 C CNN
+F 1 "12 MHz" H 2450 5800 50  0000 C CNN
+F 2 "" H 2450 5950 50  0001 C CNN
+F 3 "" H 2450 5950 50  0001 C CNN
+	1    2450 5950
+	1    0    0    -1
+$EndComp
+$Comp
+L C C?
+U 1 1 594A4B06
+P 2150 6250
+F 0 "C?" H 2175 6350 50  0000 L CNN
+F 1 "22p" H 2175 6150 50  0000 L CNN
+F 2 "" H 2188 6100 50  0001 C CNN
+F 3 "" H 2150 6250 50  0001 C CNN
+	1    2150 6250
+	1    0    0    -1
+$EndComp
+$Comp
+L C C?
+U 1 1 594A4B3A
+P 2750 6250
+F 0 "C?" H 2775 6350 50  0000 L CNN
+F 1 "22p" H 2775 6150 50  0000 L CNN
+F 2 "" H 2788 6100 50  0001 C CNN
+F 3 "" H 2750 6250 50  0001 C CNN
+	1    2750 6250
+	1    0    0    -1
+$EndComp
+$Comp
+L GND #PWR?
+U 1 1 594A4C24
+P 2450 6500
+F 0 "#PWR?" H 2450 6250 50  0001 C CNN
+F 1 "GND" H 2450 6350 50  0000 C CNN
+F 2 "" H 2450 6500 50  0001 C CNN
+F 3 "" H 2450 6500 50  0001 C CNN
+	1    2450 6500
+	1    0    0    -1
+$EndComp
+Wire Wire Line
+	2500 3950 2600 3950
+Wire Wire Line
+	2600 3950 2600 4050
+Wire Wire Line
+	2500 3650 2600 3650
+Wire Wire Line
+	2600 3650 2600 3500
+Wire Wire Line
+	2500 3850 2700 3850
+Wire Wire Line
+	2500 3750 2700 3750
+Wire Wire Line
+	2700 5500 2400 5500
+Wire Wire Line
+	2700 5400 2400 5400
+Wire Wire Line
+	2300 5950 2150 5950
+Wire Wire Line
+	2150 5950 2150 6100
+Wire Wire Line
+	2600 5950 2750 5950
+Wire Wire Line
+	2750 5950 2750 6100
+Wire Wire Line
+	2450 6500 2450 6450
+Wire Wire Line
+	2150 6450 2750 6450
+Wire Wire Line
+	2150 6450 2150 6400
+Wire Wire Line
+	2750 6450 2750 6400
+Connection ~ 2450 6450
+Wire Wire Line
+	2250 5950 2250 5600
+Wire Wire Line
+	2250 5600 2700 5600
+Connection ~ 2250 5950
+Wire Wire Line
+	2700 5700 2650 5700
+Wire Wire Line
+	2650 5700 2650 5950
+Connection ~ 2650 5950
 $EndSCHEMATC

Commit message: Desarrollo del conversor USB-UART terminado
Parts:
- added C?: 10n, symbol C
- added Q? (x2): S8050, TO-92, symbol S8050
- added R? (x2): 470, symbol R_Small
- added R? (x2): 10k, symbol R
Connections:
- net labels added: 3.3V, 5V, DTR, GPIO0, RTS, RXD, TXD
- wire segments 20 -> 57
- no-connect marks 0 -> 5
Other:
- moved on the sheet: C?, U?, Y?
