File: SLAMP-WiFi/SLAMP-WiFi.kicad_pcb (KiCad board)
At the start: 2 copper layers, 0 parts

Commit message: layout terminado
Parts:
- added C1: 1u, Capacitors_SMD:C_0805, F.Cu at (190.6, 89.3)
- added C10: 470p, Capacitors_SMD:C_0805, F.Cu at (179.6, 67.8)
- added C2: 22p, Capacitors_SMD:C_0805, F.Cu at (151.6, 95.1)
- added C3: 100n, Capacitors_SMD:C_0805, F.Cu at (152.0, 87.0)
- added C4: 22p, Capacitors_SMD:C_0805, F.Cu at (166.4, 90.9)
- added C5: 470p, Capacitors_SMD:C_0805, F.Cu at (195.1, 89.9)
- added C6: 1000uF /6.3V, Capacitors_THT:CP_Radial_D8.0mm_P3.50mm, F.Cu at (152.1, 75.2)
- added C7: 100n, Capacitors_SMD:C_0805, F.Cu at (195.1, 84.8)
- added C8: 1u, Capacitors_SMD:C_0805, F.Cu at (195.1, 87.4)
- added C9: 100nF, Capacitors_SMD:C_1210, F.Cu at (186.2, 88.5)
- added D1: LED, LEDs:LED_0805, F.Cu at (181.5, 89.5)
- added G***: LOGO, mod:wifilogo, F.Cu at (160.9, 63.8)
- added P1: POWER_IN 5V, Connectors_Terminal_Blocks:TerminalBlock_Pheonix_MKDS1.5-2pol, F.Cu at (152.1, 64.3)
- added P10: FACE5, Connectors_JST:JST_XH_B03B-XH-A_03x2.50mm_Straight, F.Cu at (174.6, 104.3)
- added P2: USB_BUS, Pin_Headers:Pin_Header_Angled_1x04_Pitch2.54mm, F.Cu at (148.8, 92.2)
- added P3: VUSB, Pin_Headers:Pin_Header_Straight_1x01, F.Cu at (151.9, 82.7)
- added P4: EXTRA, Connectors_JST:JST_XH_B03B-XH-A_03x2.50mm_Straight, F.Cu at (149.5, 104.3)
- added P5: ADC, Connectors_JST:JST_XH_B03B-XH-A_03x2.50mm_Straight, F.Cu at (158.0, 104.3)
- added P6: FACE1, Connectors_JST:JST_XH_B03B-XH-A_03x2.50mm_Straight, F.Cu at (200.2, 104.3)
- added P7: FACE2, Connectors_JST:JST_XH_B03B-XH-A_03x2.50mm_Straight, F.Cu at (191.4, 104.3)
- added P8: FACE3, Connectors_JST:JST_XH_B03B-XH-A_03x2.50mm_Straight, F.Cu at (183.0, 104.3)
- added P9: FACE4, Connectors_JST:JST_XH_B03B-XH-A_03x2.50mm_Straight, F.Cu at (166.5, 104.3)
- added Q1: S8050, TO_SOT_Packages_SMD:SOT-23, F.Cu at (158.9, 76.8)
- added Q2: S8050, TO_SOT_Packages_SMD:SOT-23, F.Cu at (162.7, 76.8)
- added R1: 470, Resistors_SMD:R_0805, F.Cu at (167.6, 83.9)
- added R10: 470, Resistors_SMD:R_0805, F.Cu at (191.4, 95.0)
- added R11: 470, Resistors_SMD:R_0805, F.Cu at (183.0, 95.0)
- added R12: 470, Resistors_SMD:R_0805, F.Cu at (166.5, 95.1)
- added R13: 220k, Resistors_SMD:R_0805, F.Cu at (181.5, 85.0)
- added R14: 100k, Resistors_SMD:R_0805, F.Cu at (186.2, 84.8)
- added R15: 470, Resistors_SMD:R_0805, F.Cu at (181.5, 87.4)
- added R16: 470, Resistors_SMD:R_0805, F.Cu at (179.6, 70.1)
- added R17: 10k, Resistors_SMD:R_0805, F.Cu at (162.7, 80.0)
- added R18: 10k, Resistors_SMD:R_0805, F.Cu at (158.4, 80.0)
- added R19: 0 (NC), Resistors_SMD:R_0805, F.Cu at (179.7, 63.4)
- added R2: 470, Resistors_SMD:R_0805, F.Cu at (167.6, 86.5)
- added R20: 470, Resistors_SMD:R_0805, F.Cu at (178.8, 75.8)
- added R3: 470, Resistors_SMD:R_0805, F.Cu at (174.6, 95.0)
- added R4: 10k, Resistors_SMD:R_0805, F.Cu at (162.7, 73.8)
- added R5: 10k, Resistors_SMD:R_0805, F.Cu at (166.5, 93.0)
- added R6: 10k, Resistors_SMD:R_0805, F.Cu at (166.2, 73.8)
- added R7: 10k, Resistors_SMD:R_0805, F.Cu at (179.7, 65.5)
- added R8: 10k, Resistors_SMD:R_0805, F.Cu at (199.0, 82.3)
- added R9: 470, Resistors_SMD:R_0805, F.Cu at (200.2, 95.0)
- added SW1: KEY_RST, Buttons_Switches_THT:SW_PUSH_6mm, F.Cu at (169.4, 63.2)
- added SW2: KEY_FLASH, Buttons_Switches_THT:SW_PUSH_6mm, F.Cu at (176.0, 76.8)
- added U1: MIC5219-3.3BM5, TO_SOT_Packages_SMD:SOT-23-5, F.Cu at (190.6, 85.7)
- added U2: CH340G, SMD_Packages:SO-16-N, F.Cu at (159.0, 86.6)
- added U3: ESP-12F, ESP8266:ESP-12E, F.Cu at (184.7, 63.4)
- added Y1: 12 MHz, Crystals:HC-49V, F.Cu at (156.5, 93.6)
Routing:
- net 5V: track 0.00 -> 121.2 mm, vias 0 -> 2
- net 3.3V: track 0.00 -> 97.5 mm, vias 0 -> 4
- net GND: track 0.00 -> 61.6 mm, vias 0 -> 2
- net EXTRA: track 0.00 -> 59.2 mm, vias 0 -> 3
- net Net-(R12-Pad2): track 0.00 -> 53.1 mm, vias 0 -> 2
- net RXD: track 0.00 -> 49.4 mm, vias 0 -> 2
- net TXD: track 0.00 -> 45.4 mm, vias 0 -> 2
- net GPIO16: track 0.00 -> 45.3 mm, vias 0 -> 7
- net Net-(R11-Pad2): track 0.00 -> 40.6 mm
- net Net-(R10-Pad2): track 0.00 -> 36.5 mm
- net Net-(R9-Pad2): track 0.00 -> 33.3 mm
- net ANALOG: track 0.00 -> 31.9 mm, vias 0 -> 2
- net Net-(R3-Pad1): track 0.00 -> 30.7 mm
- net ADC: track 0.00 -> 28.8 mm, vias 0 -> 2
- net GPIO0: track 0.00 -> 25.0 mm, vias 0 -> 2
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- added copper zone on B.Cu, net GND
- added copper zone on F.Cu, net GND
Other:
- board outline added: 61.6 x 47.2 mm
